File: pcb/badge-main/Edge-AI-Badge_Main.kicad_pcb (KiCad board)
At the start: 2 copper layers, 78 x 78 mm, 136 parts, among them J1 USB C 2.0, J2 I2C, J3 JST PH, J4 I2C, J5 UART, J6 I2C, M1 Z3OC1T8219731, Q1 DMN2058U, Q2 MMBT3904, Q3 DMN2058U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

Commit message: delete USB inversion, add diode, idk
Parts:
- removed D1: D_Schottky, Diode_SMD:D_SOD-523
- removed Q2: MMBT3904, Package_TO_SOT_SMD:SOT-23
- removed R22: 47K, Resistor_SMD:R_0402_1005Metric
- removed R23: 100K, Resistor_SMD:R_0402_1005Metric
- removed R48: 0, Resistor_SMD:R_0402_1005Metric
Routing:
- net Net-(D1-K): track 4.91 -> 0.00 mm
- net VBUS: track 12.7 -> 10.3 mm
- net Net-(Q2-B): track 1.73 -> 0.00 mm
- net SYSOFF: track 80.0 -> 79.3 mm

Commit message: some sch + pcb changes ...
Parts:
- removed R34: 10K, Resistor_SMD:R_0402_1005Metric
- added D1: MBR0540, Diode_SMD:D_SOD-123, B.Cu at (4.34, 24.4)
- C3, C4: value 0.1uF -> 12pF
- moved C19 2.12 mm to (5.92, 21.8), turned to -90 degrees
- moved TP1 1.66 mm to (4.33, 22.5)
- moved TP6 1.26 mm to (5.92, 20.0)
- moved TP5 0.13 mm to (5.46, 29.1)
Connections:
- D10 pad 4: VBUS -> VBUS_IN
- J1 pad A4: VBUS -> VBUS_IN
- J1 pad A9: VBUS -> VBUS_IN
- J1 pad B4: VBUS -> VBUS_IN
- J1 pad B9: VBUS -> VBUS_IN
Routing:
- net VBUS: track 10.3 -> 4.23 mm
- net SYSOFF: track 79.3 -> 73.5 mm
- net VBUS_IN: track 0.00 -> 4.98 mm
- net GND: track 83.2 -> 86.1 mm, vias 390 -> 391
- net +3V3: track 442.7 -> 440.4 mm
- net +BATT: track 78.3 -> 79.2 mm
- added copper zone on B.Cu, net VBUS_IN
