File: pcb/badge-main/Edge-AI-Badge_Main.kicad_sch (KiCad schematic)
At the start: 135 parts, among them J1 USB C 2.0, J2 I2C, J3 JST PH, J4 I2C, J5 UART, J6 I2C, M1 Z3OC1T8219731, Q1 DMN2058U, Q2 MMBT3904, Q3 DMN2058U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

Commit message: delete USB inversion, add diode, idk
Parts:
- removed Q2: MMBT3904, Package_TO_SOT_SMD:SOT-23, symbol Transistor_BJT:MMBT3904
- removed R22: 47K, Resistor_SMD:R_0402_1005Metric, symbol Device:R
- removed R23: 100K, Resistor_SMD:R_0402_1005Metric, symbol Device:R
- removed R48: 0, Resistor_SMD:R_0402_1005Metric, symbol Device:R
- C3, C4: value 0.1uF -> 12pF
- D1: value D_Schottky -> DSS24; footprint Diode_SMD:D_SOD-523 -> (none); LCSC C917006 -> (none)
Connections:
- net SYSOFF: no longer D1.2 (A)
- net VBUS: now also D1.1 (K); no longer D10.4 (VCC), J1.A4 (VBUS), J1.A9 (VBUS), J1.B4 (VBUS), J1.B9 (VBUS)
- new net VBUS_IN: D1.2 (A), D10.4 (VCC), J1.A4 (VBUS), J1.A9 (VBUS), J1.B4 (VBUS), J1.B9 (VBUS)
Other:
- note removed: "SYSOFF: HIGH = OFF LOW = ON"
- note removed: "invert + detect usb"
- moved on the sheet: D10

Commit message: some sch + pcb changes ...
Parts:
- removed D1: DSS24, symbol Device:D_Schottky
- removed R34: 10K, Resistor_SMD:R_0402_1005Metric, symbol Device:R
- added D1: MBR0540, Diode_SMD:D_SOD-123, symbol Diode:MBR0540
Connections:
- net VBUS: now also D1.1 (K)
- net VBUS_IN: now also D1.2 (A)
Other:
- moved on the sheet: D10, J1, R10, R9
